File: DS1339B_RTC_breakout.sch (EAGLE design)
At the start: 8 parts, among them Y1 CRYSTAL.ABS25

Commit message: added information
Other:
- note added: "I2C address: 0xd0"
- note added: "William Laney"
Changed lines of the file:
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@@
 <part name="R3" library="microbuilder" deviceset="RESISTOR" device="0805_NOOUTLINE" value="10K"/>
 <part name="+3V2" library="supply1" deviceset="+3V3" device=""/>
+<part name="FRAME1" library="frames" deviceset="A4L-LOC" device=""/>
 </parts>
 <sheets>
 <sheet>
 <plain>
+<text x="66.04" y="33.02" size="1.27" layer="97">I2C address: 0xd0</text>
+<text x="162.56" y="-22.86" size="1.6764" layer="97">William Laney</text>
 </plain>
 <instances>
@@
 <instance part="R3" gate="G$1" x="127" y="45.72" rot="R270"/>
 <instance part="+3V2" gate="G$1" x="127" y="35.56" rot="R180"/>
+<instance part="FRAME1" gate="G$1" x="-55.88" y="-43.18"/>
 </instances>
 <busses>

Commit message: intial layout of breakout board
Connections:
- removed net SDA1: R3.1
- net N$1: now also Y1.1; no longer Y1.2
- net N$2: now also Y1.2; no longer Y1.1
- net SQW/INT: now also R3.1
Other:
- moved on the sheet: Y1
Changed lines of the file:
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@@
 <setting verticaltext="up"/>
 </settings>
-<grid distance="0.1" unitdist="inch" unit="inch" style="lines" multiple="1" display="yes" altdistance="0.01" altunitdist="inch" altunit="inch"/>
+<grid distance="0.1" unitdist="inch" unit="inch" style="lines" multiple="1" display="no" altdistance="0.01" altunitdist="inch" altunit="inch"/>
 <layers>
 <layer number="1" name="Top" color="4" fill="1" visible="no" active="no"/>
@@
 <instances>
 <instance part="U$1" gate="G$1" x="76.2" y="50.8"/>
-<instance part="Y1" gate="G$1" x="53.34" y="58.42" rot="R90"/>
+<instance part="Y1" gate="G$1" x="53.34" y="58.42" rot="R270"/>
 <instance part="GND1" gate="1" x="43.18" y="38.1" rot="R270"/>
 <instance part="BAT1" gate="G$1" x="53.34" y="45.72" rot="R180"/>
@@
 </busses>
 <nets>
-<net name="N$1" class="0">
-<segment>
-<pinref part="U$1" gate="G$1" pin="X1"/>
-<pinref part="Y1" gate="G$1" pin="2"/>
-<wire x1="60.96" y1="60.96" x2="53.34" y2="60.96" width="0.1524" layer="91"/>
-</segment>
-</net>
 <net name="N$2" class="0">
 <segment>
-<pinref part="Y1" gate="G$1" pin="1"/>
-<wire x1="53.34" y1="55.88" x2="53.34" y2="53.34" width="0.1524" layer="91"/>
 <pinref part="U$1" gate="G$1" pin="X2"/>
 <wire x1="53.34" y1="53.34" x2="60.96" y2="53.34" width="0.1524" layer="91"/>
+<pinref part="Y1" gate="G$1" pin="2"/>
+<wire x1="53.34" y1="53.34" x2="53.34" y2="55.88" width="0.1524" layer="91"/>
 </segment>
 </net>
@@
 <segment>
 <pinref part="U$1" gate="G$1" pin="SQW/INT"/>
-<wire x1="91.44" y1="53.34" x2="132.08" y2="53.34" width="0.1524" layer="91"/>
+<wire x1="91.44" y1="53.34" x2="127" y2="53.34" width="0.1524" layer="91"/>
 <label x="132.08" y="53.34" size="1.27" layer="95" xref="yes"/>
+<pinref part="R3" gate="G$1" pin="1"/>
+<wire x1="127" y1="53.34" x2="132.08" y2="53.34" width="0.1524" layer="91"/>
+<wire x1="127" y1="50.8" x2="127" y2="53.34" width="0.1524" layer="91"/>
+<junction x="127" y="53.34"/>
 </segment>
 <segment>
@@
 </segment>
 </net>
-<net name="SDA1" class="0">
-<segment>
-<pinref part="R3" gate="G$1" pin="1"/>
-<wire x1="127" y1="53.34" x2="127" y2="50.8" width="0.1524" layer="91"/>
-</segment>
-</net>
+<net name="N$1" class="0">
+<segment>
+<pinref part="Y1" gate="G$1" pin="1"/>
+<pinref part="U$1" gate="G$1" pin="X1"/>
+<wire x1="53.34" y1="60.96" x2="60.96" y2="60.96" width="0.1524" layer="91"/>
+</segment>
+</net>
