File: DS1339B_RTC_breakout.brd (EAGLE design)
At the start: 22.9 x 15.2 mm, 8 parts, among them Y1 CRYSTAL.ABS25

Commit message: added silk screen
Routing:
- net +3V3: track 33.3 -> 32.3 mm
Other:
- board text added: "0.1uF"
- board text added: "10k"
- board text added: "ABS25"
- board text added: "DS1339B"
- board text added: "DS1339B Breakout v1"
- board text added: "GND"
- board text added: "SCL"
- board text added: "SDA"
- board text added: "SQW"
- board text added: "VCC"
- board text added: "VIMS"
- board text added: "WM Physics"
- board text added: "William Laney 2016"
